Commit message: synced v2

File: pybullet/ball.urdf (robot description, URDF)
Before this commit: robot plosca, 1 links, 0 joints
Links:
- link ball: mass 0.01 -> 0.002456

File: pybullet/plosca.urdf (robot description, URDF)
Before this commit: robot plosca, 3 links, 2 joints
Links:
- link base_link: mass None -> 1
- link zgornja_plosca: mass None -> 3; geometry collision cylinder length=0.004 radius=0.18; visual cylinder length=0.004 radius=0.18

Commit message: successful RL balancing with TD3

File: pybullet/ball.urdf (robot description, URDF)
Before this commit: robot plosca, 1 links, 0 joints
Links:
- link ball: mass 0.002456 -> 0.015
